Commit message: Changes to gripper

File: niryo_one_description/urdf/bot.xacro (robot description, xacro)
@@ -2,8 +2,6 @@
   <robot xmlns:xacro="http://ros.org/wiki/xacro">
   <xacro:macro name="bot" params="prefix parent name *origin">
-    <!--
     <xacro:include filename="$(find niryo_one_description)/urdf/niryo_one_gripper.urdf.xacro"/>
     <xacro:gripper prefix="${prefix}"/>
-    -->
     <xacro:property name="distance_origin_shoulder_z" value="0.103" />
     <xacro:property name="distance_shoulder_arm_z" value="0.080" />

File: niryo_one_description/urdf/niryo_one_gripper.urdf.xacro (robot description, xacro)
@@ -30,5 +30,5 @@
             <geometry>
                 <mesh
-                        filename="package://niryo_robot_description/meshes/gripper_1/base_gripper_1.STL"/>
+                        filename="package://niryo_one_description/meshes/gripper_1/base_gripper_1.STL"/>
             </geometry>
         </visual>
@@ -38,5 +38,5 @@
             <geometry>
                 <mesh
-                        filename="package://niryo_robot_description/meshes/gripper_1/base_gripper_1.STL"/>
+                        filename="package://niryo_one_description/meshes/gripper_1/base_gripper_1.STL"/>
             </geometry>
         </collision>
@@ -62,5 +62,5 @@
             <geometry>
                 <mesh
-                        filename="package://niryo_robot_description/meshes/gripper_1/mors_1.STL"/>
+                        filename="package://niryo_one_description/meshes/gripper_1/mors_1.STL"/>
             </geometry>
             <material name="">
@@ -73,5 +73,5 @@
             <geometry>
                 <mesh
-                        filename="package://niryo_robot_description/meshes/gripper_1/mors_1.STL"/>
+                        filename="package://niryo_one_description/meshes/gripper_1/mors_1.STL"/>
             </geometry>
         </collision>
@@ -89,4 +89,5 @@
                effort="1"
                velocity="5"/>
+        <mimic joint="${prefix}_gripper_joint" multiplier="1" offset="0" />
     </joint>
     <!-- Mors 2 -->
@@ -110,5 +111,5 @@
             <geometry>
                 <mesh
-                        filename="package://niryo_robot_description/meshes/gripper_1/mors_2.STL"/>
+                        filename="package://niryo_one_description/meshes/gripper_1/mors_2.STL"/>
             </geometry>
         </visual>
@@ -118,5 +119,5 @@
             <geometry>
                 <mesh
-                        filename="package://niryo_robot_description/meshes/gripper_1/mors_2.STL"/>
+                        filename="package://niryo_one_description/meshes/gripper_1/mors_2.STL"/>
             </geometry>
         </collision>
@@ -133,5 +134,17 @@
                effort="1"
                velocity="5"/>
+        <mimic joint="${prefix}_joint_base_to_mors_1" multiplier="1" offset="0" />
     </joint>
+    <ros2_control name="${prefix}_gripper" type="actuator">
+      <hardware>
+        <plugin>niryo_one_driver/NiryoOneActuatorInterface</plugin>
+      </hardware>
+      <joint name="${prefix}_joint_base_to_mors_1">
+        <command_interface name="position"/>
+        <state_interface name="position"/>
+        <state_interface name="velocity"/>
+        <state_interface name="effort"/>
+      </joint>
+    </ros2_control>
     <xacro:macro name="SimpleTransmissionEffort" params="joint n">
     <transmission name="${prefix}_transmission_${n}">
