Commit message: fixed error in gripper urdf

File: niryo_one_description/urdf/niryo_one_gripper.urdf.xacro (robot description, xacro)
@@ -89,5 +89,4 @@
                effort="1"
                velocity="5"/>
-        <mimic joint="${prefix}_gripper_joint" multiplier="1" offset="0" />
     </joint>
     <!-- Mors 2 -->
